Commit message: rename and only publish join

File: articubot_one/description/robot_core.xacro (robot description, xacro)
@@ -50,6 +50,6 @@
         <parent link="chassis"/>
         <child link="laser_frame"/>
-        <origin xyz="0.1 0 0.175" rpy="0 0 0"/>
-        <axis rpy="0 0 0" xyz="0 1 0" />
+        <origin xyz="0.1 0 0.175" rpy="0 0 -${1.5*pi}"/>
+        <axis rpy="0 0 0" xyz="1 0 0" />
         <limit effort="0.1" lower="-0.6" upper="0.6" velocity="0.2"/>
     </joint>

Commit message: working 3d scan

File: articubot_one/description/robot_core.xacro (robot description, xacro)
@@ -50,5 +50,6 @@
         <parent link="chassis"/>
         <child link="laser_frame"/>
-        <origin xyz="0.1 0 0.175" rpy="0 0 -${1.5*pi}"/>
+        <!-- <origin xyz="0.1 0 0.175" rpy="0 0 -${1.5*pi}"/> -->
+        <origin xyz="0.1 0 0.175" rpy="0 0 0"/>
         <axis rpy="0 0 0" xyz="1 0 0" />
         <limit effort="0.1" lower="-0.6" upper="0.6" velocity="0.2"/>
